File: ergogen/output/pcbs/prototype_routed.kicad_pcb (KiCad board)
At the start: 2 copper layers, 136.1 x 97.6 mm, 49 parts

Commit message: feat: updated PCB
Parts:
- added Asuka: LOGO, LOGO, F.Cu at (204.8, 174.2)
- added Rei: LOGO, LOGO, B.Cu at (205.7, 172.3)
- moved LOGO1 129.3 mm to (284.2, 127.0)
- moved S11 78.0 mm to (206.0, 126.7)
- moved S3 78.0 mm to (149.0, 122.7)
- moved D17 78.0 mm to (244.0, 139.2)
- moved D2 78.0 mm to (149.0, 146.7)
- moved MH1 78.0 mm to (158.5, 151.2)
- moved D12 78.0 mm to (206.0, 112.7)
- moved D4 78.0 mm to (168.0, 165.7)
- moved D5 78.0 mm to (168.0, 146.7)
- moved S18 78.0 mm to (244.0, 115.2)
- moved S19 78.0 mm to (227.0, 172.7)
- moved S6 78.0 mm to (168.0, 122.7)
- moved S2 78.0 mm to (149.0, 141.7)
- moved S5 78.0 mm to (168.0, 141.7)
- moved S8 78.0 mm to (187.0, 136.7)
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Routing:
- net space_cluster: track 44.1 -> 44.9 mm
